File: IGEM_Device.sch (KiCad schematic (older format))
At the start: 12 parts, among them J1 67997-410HLF, Q1 MMBT3906, U1 SaBLE-X-R2, U2 TC1014-2.85VCT713, U3 LMP91000SD_NOPB

Commit message: version 1 s Please enter the commit message for your changes. Lines starting
Parts:
- added C4: 0.1u, symbol Device:C
- added C5: 0.47u, symbol Device:C
- added R4: 100k, symbol Device:R
- added U5: TPS79718QDCKRQ1, DCK5, symbol IGEM_Device:TPS79718QDCKRQ1
- gave numbers to parts that had none: 1
Connections:
- net +2V85: now also C4.1, U5.4 (IN)
- net GND: now also C4.2, C5.2, U5.2 (GND)
- net POWER_GOOD: now reaches U1.21 (DIO_8)
- net POWER_GOOD: now also R4.2, U5.1 (PG)
- net +1V8: now reaches U3.11 (VREF)
- net +1V8: now also C5.1, R4.1, U5.5 (OUT)
- net IP_ANODE: now reaches R3.1, U4.2 (R)
- net IP_CATHODE: now reaches Q1.3 (C)
- no-connect marks 16 -> 17
Other:
- moved on the sheet: J1, R1, R2, U1, U3
