File: IGEM_Device.sch (KiCad schematic (older format))
At the start: 16 parts, among them J1 67997-410HLF, Q1 MMBT3906, U1 SaBLE-X-R2, U2 TC1014-2.85VCT713, U3 LMP91000SD_NOPB, U4 LM334MX_NOPB, U5 TPS79718QDCKRQ1

Commit message: version 2
Parts:
- removed Q1: MMBT3906, Package_TO_SOT_SMD:SOT-23, symbol Transistor_BJT:MMBT3906
- added D1: 1N4148, Diode_THT:D_DO-35_SOD27_P7.62mm_Horizontal, symbol Diode:1N4148
- added R5: 909, symbol Device:R
- R3: value 84.5 -> 90.9
Connections:
- net GND: no longer R3.2, U4.1 (V-)
- net IP_CATHODE: now also R3.2, U4.2 (R), R5.2
- net IP_CONTROL: now reaches U1.17 (DIO_2)
- net IP_CONTROL: now also U4.3 (V+)
- net IP_ANODE: no longer names the net of R3.1
- net IP_ANODE: now also U4.1 (V-), D1.2 (A); no longer U4.2 (R)
- new net: D1.1 (K), R5.1
Changed lines of the file:
@@
 	1    0    0    -1
 $EndComp
-$Comp
-L IGEM_Device:+2V85 #PWR?
-U 1 1 5CF7974B
-P 5350 4250
-F 0 "#PWR?" H 5350 4100 50  0001 C CNN
-F 1 "+2V85" H 5365 4423 50  0000 C CNN
-F 2 "" H 5350 4250 50  0001 C CNN
-F 3 "" H 5350 4250 50  0001 C CNN
-	1    5350 4250
-	1    0    0    -1
-$EndComp
-$Comp
-L power:GND #PWR?
-U 1 1 5CF7DBF5
-P 6000 5650
-F 0 "#PWR?" H 6000 5400 50  0001 C CNN
-F 1 "GND" H 6005 5477 50  0000 C CNN
-F 2 "" H 6000 5650 50  0001 C CNN
-F 3 "" H 6000 5650 50  0001 C CNN
-	1    6000 5650
-	1    0    0    -1
-$EndComp
-Wire Wire Line
-	6300 4900 6000 4900
-Wire Wire Line
-	6000 4900 6000 5550
 NoConn ~ 6300 5200
 NoConn ~ 7650 5200
@@
 NoConn ~ 7650 5000
 NoConn ~ 7650 4900
-$Comp
-L Device:R R3
-U 1 1 5CF92324
-P 6150 5350
-F 0 "R3" H 6220 5396 50  0000 L CNN
-F 1 "84.5" H 6220 5305 50  0000 L CNN
-F 2 "" V 6080 5350 50  0001 C CNN
-F 3 "~" H 6150 5350 50  0001 C CNN
-	1    6150 5350
-	1    0    0    -1
-$EndComp
-Wire Wire Line
-	6300 5000 6150 5000
-Wire Wire Line
-	6150 5000 6150 5200
-Wire Wire Line
-	6150 5500 6150 5550
-Wire Wire Line
-	6150 5550 6000 5550
-$Comp
-L Transistor_BJT:MMBT3906 Q1
-U 1 1 5CF9C096
-P 5450 4500
-F 0 "Q1" H 5640 4454 50  0000 L CNN
-F 1 "MMBT3906" H 5640 4545 50  0000 L CNN
-F 2 "Package_TO_SOT_SMD:SOT-23" H 5650 4425 50  0001 L CIN
-F 3 "https://www.fairchildsemi.com/datasheets/2N/2N3906.pdf" H 5450 4500 50  0001 L CNN
-	1    5450 4500
-	-1   0    0    1
-$EndComp
-Wire Wire Line
-	6000 5550 6000 5650
-Connection ~ 6000 5550
-Wire Wire Line
-	5350 4250 5350 4300
-Wire Wire Line
-	6300 5100 5800 5100
-Wire Wire Line
-	5800 4500 5650 4500
-Wire Wire Line
-	5800 4500 5800 5100
 Text Label 8800 1350 2    50   ~ 0
 TEMP_OUT
@@
 Wire Wire Line
 	4550 3100 4550 3650
-Text Label 4800 4850 0    50   ~ 0
+$Comp
+L Device:R R3
+U 1 1 5CFD9641
+P 5850 4800
+F 0 "R3" H 5920 4846 50  0000 L CNN
+F 1 "90.9" H 5920 4755 50  0000 L CNN
+F 2 "" V 5780 4800 50  0001 C CNN
+F 3 "~" H 5850 4800 50  0001 C CNN
+	1    5850 4800
+	1    0    0    -1
+$EndComp
+$Comp
+L Device:R R5
+U 1 1 5CFD9695
+P 5400 4800
+F 0 "R5" H 5470 4846 50  0000 L CNN
+F 1 "909" H 5470 4755 50  0000 L CNN
+F 2 "" V 5330 4800 50  0001 C CNN
+F 3 "~" H 5400 4800 50  0001 C CNN
+	1    5400 4800
+	1    0    0    -1
+$EndComp
+$Comp
+L Diode:1N4148 D1
+U 1 1 5CFD974D
+P 5700 4550
+F 0 "D1" H 5700 4766 50  0000 C CNN
+F 1 "1N4148" H 5700 4675 50  0000 C CNN
+F 2 "Diode_THT:D_DO-35_SOD27_P7.62mm_Horizontal" H 5700 4375 50  0001 C CNN
+F 3 "http://www.nxp.com/documents/data_sheet/1N4148_1N4448.pdf" H 5700 4550 50  0001 C CNN
+	1    5700 4550
+	1    0    0    -1
+$EndComp
+Wire Wire Line
+	6300 5000 5850 5000
+Wire Wire Line
+	5850 5000 5850 4950
+Wire Wire Line
+	6300 4900 6300 4550
+Wire Wire Line
+	6300 4550 5850 4550
+Wire Wire Line
+	5850 4550 5850 4650
+Connection ~ 5850 4550
+Wire Wire Line
+	5550 4550 5400 4550
+Wire Wire Line
+	5400 4550 5400 4650
+Wire Wire Line
+	5400 4950 5400 5000
+Wire Wire Line
+	5400 5000 5850 5000
+Connection ~ 5850 5000
+Text Label 4800 5000 0    50   ~ 0
 IP_CATHODE
-Text Label 4800 5000 0    50   ~ 0
-IP_ANODE
-Wire Wire Line
-	5350 4700 5350 4850
-Wire Wire Line
-	5350 4850 4800 4850
-Wire Wire Line
-	6150 5000 4800 5000
-Connection ~ 6150 5000
+Wire Wire Line
+	5400 5000 4800 5000
+Connection ~ 5400 5000
+Text Label 5800 5100 0    50   ~ 0
+IP_CONTROL
+Wire Wire Line
+	6300 5100 5800 5100
+Text Label 4150 3600 1    50   ~ 0
+IP_CONTROL
+Wire Wire Line
+	4150 3100 4150 3600
 $EndSCHEMATC
